Commit message: tuning pid

File: reachy_moveit.urdf (robot description, URDF)
Before this commit: robot reachy, 21 links, 20 joints
Joints:
- joint l_arm_yaw: limit lower=-1.57 upper=1.57 effort=100.0 velocity=100.0 -> lower=-1.57 upper=1.57 effort=1000.0 velocity=1000.0
- joint l_elbow_pitch: limit lower=-2.182 upper=0 effort=100.0 velocity=100.0 -> lower=-2.182 upper=0 effort=1000.0 velocity=1000.0
- joint l_forearm_yaw: limit lower=-1.745 upper=1.745 effort=100.0 velocity=100.0 -> lower=-1.745 upper=1.745 effort=1000.0 velocity=1000.0
- joint l_gripper: limit lower=-0.35 upper=1.2 effort=100.0 velocity=100.0 -> lower=-0.35 upper=1.2 effort=1000.0 velocity=1000.0
- joint l_shoulder_pitch: limit lower=-2.618 upper=1.57 effort=100.0 velocity=100.0 -> lower=-2.618 upper=1.57 effort=1000.0 velocity=1000.0
- joint l_shoulder_roll: limit lower=-0.174 upper=3.14 effort=100.0 velocity=100.0 -> lower=-0.174 upper=3.14 effort=1000.0 velocity=1000.0
- joint l_wrist_pitch: limit lower=-0.785 upper=0.785 effort=100.0 velocity=100.0 -> lower=-0.785 upper=0.785 effort=1000.0 velocity=1000.0
- joint l_wrist_roll: limit lower=-0.785 upper=0.785 effort=100.0 velocity=100.0 -> lower=-0.785 upper=0.785 effort=1000.0 velocity=1000.0
- joint r_arm_yaw: limit lower=-1.57 upper=1.57 effort=100.0 velocity=100.0 -> lower=-1.57 upper=1.57 effort=1000.0 velocity=1000.0
- joint r_elbow_pitch: limit lower=-2.182 upper=0 effort=100.0 velocity=100.0 -> lower=-2.182 upper=0 effort=1000.0 velocity=1000.0
- joint r_forearm_yaw: limit lower=-1.745 upper=1.745 effort=100.0 velocity=100.0 -> lower=-1.745 upper=1.745 effort=1000.0 velocity=1000.0
- joint r_gripper: limit lower=-1.2 upper=0.35 effort=100.0 velocity=100.0 -> lower=-1.2 upper=0.35 effort=1000.0 velocity=1000.0
- joint r_shoulder_pitch: limit lower=-2.618 upper=1.57 effort=10.0 velocity=100.0 -> lower=-2.618 upper=1.57 effort=10.0 velocity=1000.0
- joint r_shoulder_roll: limit lower=-3.14 upper=0.174 effort=100.0 velocity=100.0 -> lower=-3.14 upper=0.174 effort=1000.0 velocity=1000.0
- joint r_wrist_pitch: limit lower=-0.785 upper=0.785 effort=100.0 velocity=100.0 -> lower=-0.785 upper=0.785 effort=1000.0 velocity=1000.0
- joint r_wrist_roll: limit lower=-0.785 upper=0.785 effort=100.0 velocity=100.0 -> lower=-0.785 upper=0.785 effort=1000.0 velocity=1000.0
